File: CO2Sensor.kicad_pcb (KiCad board)
At the start: 2 copper layers, 94 x 68.6 mm, 18 parts, among them J1 Screw_Terminal_01x02, U1 ESP32_DevKit_V1_DOIT, U2 MH-Z19B

Commit message: Rotate KiCAD Logo
Parts:
- turned REF** to 180 degrees
